File: new_stuff_june_2020/slope_generators/power_supply.sch (KiCad schematic (older format))
At the start: 18 parts

Commit message: slope gen progress, misc cleanup
Parts:
- added J3: power_in, Connector_PinHeader_2.54mm:PinHeader_2x05_P2.54mm_Vertical, symbol Connector_Generic:Conn_02x05_Odd_Even
- C10, C11, C12, C13, C14, C15, C6, C7, C8, C9: renamed from C?; footprint (none) -> Capacitor_SMD:C_0805_2012Metric_Pad1.15x1.40mm_HandSolder
- C16, C17: renamed from C?; footprint (none) -> Capacitor_THT:CP_Radial_D6.3mm_P2.50mm
- U1, U2, U4, U5: renamed from U?; footprint (none) -> Package_SO:SOIC-8_3.9x4.9mm_P1.27mm
- U3, U6: renamed from U?; footprint (none) -> Package_SO:SOIC-14_3.9x8.7mm_P1.27mm
Connections:
- net +12V: now also J3.1 (Pin_1), J3.2 (Pin_2)
- net -12V: now also J3.10 (Pin_10), J3.9 (Pin_9)
- net GND: now also J3.3 (Pin_3), J3.4 (Pin_4), J3.5 (Pin_5), J3.6 (Pin_6), J3.7 (Pin_7), J3.8 (Pin_8)
