File: new_stuff_june_2020/slope_generators/slope_generator_1.sch (KiCad schematic (older format))
At the start: 76 parts

Commit message: slope gen progress, misc cleanup
Parts:
- removed C?: 47pF, symbol Device:C
- removed Q? (x3): 2N3904, Package_TO_SOT_THT:TO-92_Inline, symbol Transistor_BJT:2N3904
- removed Q? (x3): 2N3906, Package_TO_SOT_THT:TO-92_Inline, symbol Transistor_BJT:2N3906
- added Q1, Q2, Q4: MMBT3906, Package_TO_SOT_SMD:SOT-23_Handsoldering, symbol Transistor_BJT:MMBT3906
- added Q3, Q5, Q6: MMBT3904, Package_TO_SOT_SMD:SOT-23_Handsoldering, symbol Transistor_BJT:MMBT3904
- added R1: 270k, Resistor_SMD:R_0805_2012Metric_Pad1.15x1.40mm_HandSolder, symbol Device:R
- added R16, R5: 560k, Resistor_SMD:R_0805_2012Metric_Pad1.15x1.40mm_HandSolder, symbol Device:R
- added SW2: auto_cycle_switch, slope_generators:SPDT_on_on, symbol Switch:SW_SPDT
- C1, C2, C3, C4, C5: renamed from C?; footprint (none) -> Capacitor_SMD:C_0805_2012Metric_Pad1.15x1.40mm_HandSolder
- D1, D2, D3, D4, D5, D6, D7: renamed from D?; footprint (none) -> Diode_SMD:D_SOD-123
- D8: renamed from D?; footprint (none) -> LED_THT:LED_D5.0mm
- R10, R11, R12, R13, R14, R15, R17, R18, R19, R2, R20, R21, R22, R23, R24, R25, R26, R27, R28, R29, R3, R30, R31, R32, R33, R34, R35, R36, R37, R38, R39, R4, R40, R41, R42, R43, R44, R45, R6, R7, R8, R9: renamed from R?; footprint (none) -> Resistor_SMD:R_0805_2012Metric_Pad1.15x1.40mm_HandSolder
- RV1, RV2, RV3: renamed from RV?; footprint (none) -> Potentiometer_THT:Potentiometer_Alpha_RD901F-40-00D_Single_Vertical
- RV4: renamed from RV?; footprint (none) -> Potentiometer_THT:Potentiometer_Bourns_3296W_Vertical
- SW1: renamed from SW?; footprint (none) -> slope_generators:SPDT_on_on
- SW3: renamed from SW?; value center_off -> rise-fall-both-switch; footprint (none) -> slope_generators:SPDT_on_on
- U1, U2: renamed from U?; footprint (none) -> Package_SO:SOIC-8_3.9x4.9mm_P1.27mm
- U3: renamed from U?; footprint (none) -> Package_SO:SOIC-14_3.9x8.7mm_P1.27mm
Connections:
- net +12V: now also Q1.2 (E), R1.1
- net -12V: now also R16.1, R5.1
- net GND: now also Q2.3 (C), Q3.3 (C), Q6.2 (E); no longer SW1.3 (C)
- net end_out: now also SW2.3 (C)
- net fall_CV: now also Q4.1 (B)
- net rise_CV: now also Q3.1 (B), R16.2
- net at R36.1: now also Q2.2 (E), Q3.2 (E), Q4.2 (E), Q5.2 (E)
- net at R29.1, R33.1: now also Q2.1 (B), Q5.1 (B)
- net at C5.2, U2.2 (-): now also Q4.3 (C), Q5.3 (C)
- net at D5.1 (K), R27.2: now also Q1.3 (C)
- net at R23.2, R25.1: now also Q1.1 (B)
- net at R10.2, R17.1, U1.7: no longer R15.1
- net at R4.1, SW1.2 (B): now also R15.1
- net at R10.1, R4.2, U1.6 (-): now also R5.2
- net at D7.1 (K), R44.1: now also Q6.1 (B)
- net at R45.1: now also Q6.3 (C)
- net cycle_in: no longer names the net of C2.2, R7.1
- net cycle_in: now also SW2.2 (B)
- net slope_1_expo_CV_in renamed expo_CV_in
- net slope_1_in renamed gate_in
- net slope_1_out renamed slope_out
- net slope_out: now also SW1.3 (C); no longer SW1.1 (A)
- new net: R1.2, SW1.1 (A)
Other:
- note added: "adjust for\nreliable \ntriggering\nand +5v \npeak output"
- note added: "center off"
- moved on the sheet: C1, C2, C3, D1, D2, D3, D4, D5, R10, R11, R12, R15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
