File: new_stuff_june_2020/sub_osc_board/power_supply.sch (KiCad schematic (older format))
At the start: 27 parts, among them J3 Conn_02x05_Odd_Even, U1 TL072, U10 TL072, U2 TL072, U3 TL072, U4 TL072, U5 TL072, U6 TL072, U7 40106, U8 4013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

Commit message: slope gen progress, misc cleanup
Parts:
- J3: value Conn_02x05_Odd_Even -> power_input
Changed lines of the file:
@@
 AR Path="/5EE5F4A3/5EF9A242" Ref="J3"  Part="1"
 F 0 "J3" H 6150 7617 50  0000 C CNN
-F 1 "Conn_02x05_Odd_Even" H 6150 7526 50  0000 C CNN
+F 1 "power_input" H 6150 7526 50  0000 C CNN
 F 2 "Connector_PinHeader_2.54mm:PinHeader_2x05_P2.54mm_Vertical" H 6100 7200 50  0001 C CNN
 F 3 "~" H 6100 7200 50  0001 C CNN
