File: new_stuff_june_2020/sub_osc_board/sub_osc_board.sch (KiCad schematic (older format))
At the start: 25 parts, among them J1 Conn_01x05, J2 Conn_01x03, J4 Conn_01x05, J5 Conn_01x03, J6 Conn_01x03, J7 Conn_01x03, U10 TL072, U6 TL072, U9 TL072

Commit message: slope gen progress, misc cleanup
Parts:
- J1: value Conn_01x05 -> signal_inputs
- J2: value Conn_01x03 -> pwm_inputs
- J4: value Conn_01x05 -> signal_outputs
Other:
- note added: "octave 1 wave select switch\nSPDT center off"
- note added: "octave 2 wave select switch\nSPDT center off"
- note added: "octave 3 wave select switch\nSPDT center off"
Changed lines of the file:
@@
 P 1800 1150
 F 0 "J1" H 1718 1567 50  0000 C CNN
-F 1 "Conn_01x05" H 1718 1476 50  0000 C CNN
+F 1 "signal_inputs" H 1718 1476 50  0000 C CNN
 F 2 "Connector_PinHeader_2.54mm:PinHeader_1x05_P2.54mm_Vertical" H 1800 1150 50  0001 C CNN
 F 3 "~" H 1800 1150 50  0001 C CNN
@@
 P 1800 2400
 F 0 "J2" H 1718 2717 50  0000 C CNN
-F 1 "Conn_01x03" H 1718 2626 50  0000 C CNN
+F 1 "pwm_inputs" H 1718 2626 50  0000 C CNN
 F 2 "Connector_PinHeader_2.54mm:PinHeader_1x03_P2.54mm_Vertical" H 1800 2400 50  0001 C CNN
 F 3 "~" H 1800 2400 50  0001 C CNN
@@
 P 10450 5750
 F 0 "J4" H 10530 5792 50  0000 L CNN
-F 1 "Conn_01x05" H 10530 5701 50  0000 L CNN
+F 1 "signal_outputs" H 10530 5701 50  0000 L CNN
 F 2 "Connector_PinHeader_2.54mm:PinHeader_1x05_P2.54mm_Vertical" H 10450 5750 50  0001 C CNN
 F 3 "~" H 10450 5750 50  0001 C CNN
@@
 Text Label 4250 1100 2    50   ~ 0
 saw_in
+Text Notes 2650 3750 0    50   ~ 0
+octave 1 wave select switch\nSPDT center off
+Text Notes 5450 3800 0    50   ~ 0
+octave 2 wave select switch\nSPDT center off
+Text Notes 8750 3800 0    50   ~ 0
+octave 3 wave select switch\nSPDT center off
 $EndSCHEMATC
