File: new_stuff_june_2020/oscillator_carrier_board/kicad_docs/VCO_core_components.sch (KiCad schematic (older format))
At the start: 28 parts, among them J10 Conn_01x05, J4 Conn_01x04, J5 Conn_01x02, J6 Conn_01x02, J7 Conn_01x05, J8 power_header, J9 to_VCO_board, SW1 SW_Rotary12, U1 TL072

Commit message: make gerbers of most boards, add unfinished modulation source
Parts:
- added TP1, TP2: TestPoint, TestPoint:TestPoint_Keystone_5000-5004_Miniature, symbol Connector:TestPoint
- SW1: value SW_Rotary12 -> octave_switch
Connections:
- net GND: now also R7.2, TP1.1
- net at RV6.3, U1.1: now also J10.1 (Pin_1), RV6.2, TP2.1; no longer U1.2 (-)
- net at SW1.13, U1.3 (+): now also C1.1
- new net: R7.1, RV6.1, U1.2 (-)
Other:
- note added: "octave switch trim"
- moved on the sheet: C1, J8, R7, RV6, U1A
Changed lines of the file:
@@
 AR Path="/5EF50E5A/5EF665A1" Ref="SW1"  Part="1"
 F 0 "SW1" H 5550 2331 50  0000 C CNN
-F 1 "SW_Rotary12" H 5550 2240 50  0000 C CNN
+F 1 "octave_switch" H 5550 2240 50  0000 C CNN
 F 2 "kicad_docs:apha_SR2612F-0112" H 5450 2250 50  0001 C CNN
 F 3 "http://cdn-reichelt.de/documents/datenblatt/C200/DS-Serie%23LOR.pdf" H 5450 2250 50  0001 C CNN
@@
 L Device:R_POT RV?
 U 1 1 5EF66615
-P 7500 1650
+P 7750 2000
 AR Path="/5EF66615" Ref="RV?"  Part="1"
 AR Path="/5EF50E5A/5EF66615" Ref="RV6"  Part="1"
-F 0 "RV6" V 7385 1650 50  0000 C CNN
-F 1 "???" V 7500 1650 50  0000 C CNN
-F 2 "Potentiometer_THT:Potentiometer_Bourns_3296W_Vertical" H 7500 1650 50  0001 C CNN
-F 3 "~" H 7500 1650 50  0001 C CNN
-	1    7500 1650
-	0    1    -1   0
-$EndComp
-Wire Wire Line
-	7250 1650 7350 1650
-Wire Wire Line
-	7500 1500 7500 1400
-Wire Wire Line
-	7500 1400 7750 1400
-Wire Wire Line
-	7750 1400 7750 1650
-Wire Wire Line
-	7750 1650 7650 1650
+F 0 "RV6" V 7635 2000 50  0000 C CNN
+F 1 "???" V 7750 2000 50  0000 C CNN
+F 2 "Potentiometer_THT:Potentiometer_Bourns_3296W_Vertical" H 7750 2000 50  0001 C CNN
+F 3 "~" H 7750 2000 50  0001 C CNN
+	1    7750 2000
+	0    -1   1    0
+$EndComp
 $Comp
 L Device:R R?
 U 1 1 5EF66620
-P 8000 1650
+P 7350 2250
 AR Path="/5EF66620" Ref="R?"  Part="1"
 AR Path="/5EF50E5A/5EF66620" Ref="R7"  Part="1"
-F 0 "R7" V 7900 1650 50  0000 C CNN
-F 1 "???" V 8000 1650 50  0000 C CNN
-F 2 "Resistor_SMD:R_0805_2012Metric_Pad1.15x1.40mm_HandSolder" V 7930 1650 50  0001 C CNN
-F 3 "~" H 8000 1650 50  0001 C CNN
-	1    8000 1650
-	0    1    1    0
-$EndComp
-Wire Wire Line
-	7850 1650 7750 1650
-Connection ~ 7750 1650
+F 0 "R7" H 7250 2250 50  0000 C CNN
+F 1 "???" V 7350 2250 50  0000 C CNN
+F 2 "Resistor_SMD:R_0805_2012Metric_Pad1.15x1.40mm_HandSolder" V 7280 2250 50  0001 C CNN
+F 3 "~" H 7350 2250 50  0001 C CNN
+	1    7350 2250
+	1    0    0    -1
+$EndComp
 NoConn ~ 5250 1750
 NoConn ~ 5250 1850
@@
 L Connector_Generic:Conn_02x05_Odd_Even J?
 U 1 1 5EF66650
-P 8800 3050
+P 10450 4300
 AR Path="/5EF66650" Ref="J?"  Part="1"
 AR Path="/5EF50E5A/5EF66650" Ref="J8"  Part="1"
-F 0 "J8" H 8750 2600 50  0000 C CNN
-F 1 "power_header" H 8700 2700 50  0000 C CNN
-F 2 "Connector_PinSocket_2.54mm:PinSocket_2x05_P2.54mm_Vertical" H 8800 3050 50  0001 C CNN
-F 3 "~" H 8800 3050 50  0001 C CNN
-	1    8800 3050
+F 0 "J8" H 10400 3850 50  0000 C CNN
+F 1 "power_header" H 10350 3950 50  0000 C CNN
+F 2 "Connector_PinSocket_2.54mm:PinSocket_2x05_P2.54mm_Vertical" H 10450 4300 50  0001 C CNN
+F 3 "~" H 10450 4300 50  0001 C CNN
+	1    10450 4300
 	-1   0    0    1
 $EndComp
@@
 pulse_out
 Wire Wire Line
-	8500 2850 9000 2850
-Wire Wire Line
-	9000 2950 9000 3050
-Wire Wire Line
-	9000 3050 9000 3150
-Connection ~ 9000 3050
-Wire Wire Line
-	9000 3150 8500 3150
-Connection ~ 9000 3150
-Wire Wire Line
-	8500 3150 8500 3050
-Connection ~ 8500 3150
-Wire Wire Line
-	8500 3050 8500 2950
-Connection ~ 8500 3050
-Wire Wire Line
-	8500 2950 9000 2950
-Connection ~ 8500 2950
-Connection ~ 9000 2950
-Wire Wire Line
-	9000 3050 8500 3050
-Wire Wire Line
-	8500 3250 9000 3250
+	10150 4100 10650 4100
+Wire Wire Line
+	10650 4200 10650 4300
+Wire Wire Line
+	10650 4300 10650 4400
+Connection ~ 10650 4300
+Wire Wire Line
+	10650 4400 10150 4400
+Connection ~ 10650 4400
+Wire Wire Line
+	10150 4400 10150 4300
+Connection ~ 10150 4400
+Wire Wire Line
+	10150 4300 10150 4200
+Connection ~ 10150 4300
+Wire Wire Line
+	10150 4200 10650 4200
+Connection ~ 10150 4200
+Connection ~ 10650 4200
+Wire Wire Line
+	10650 4300 10150 4300
+Wire Wire Line
+	10150 4500 10650 4500
 $Comp
 L power:GND #PWR0125
 U 1 1 5EF8CA69
-P 8500 3050
-F 0 "#PWR0125" H 8500 2800 50  0001 C CNN
-F 1 "GND" V 8505 2922 50  0000 R CNN
-F 2 "" H 8500 3050 50  0001 C CNN
-F 3 "" H 8500 3050 50  0001 C CNN
-	1    8500 3050
+P 10150 4300
+F 0 "#PWR0125" H 10150 4050 50  0001 C CNN
+F 1 "GND" V 10155 4172 50  0000 R CNN
+F 2 "" H 10150 4300 50  0001 C CNN
+F 3 "" H 10150 4300 50  0001 C CNN
+	1    10150 4300
 	0    1    1    0
 $EndComp
@@
 L Device:C C1
 U 1 1 5EFA493B
-P 8350 1800
-F 0 "C1" H 8465 1846 50  0000 L CNN
-F 1 "100nF" H 8465 1755 50  0000 L CNN
-F 2 "Capacitor_SMD:C_0805_2012Metric_Pad1.15x1.40mm_HandSolder" H 8388 1650 50  0001 C CNN
-F 3 "~" H 8350 1800 50  0001 C CNN
-	1    8350 1800
+P 6400 1700
+F 0 "C1" H 6515 1746 50  0000 L CNN
+F 1 "100nF" H 6515 1655 50  0000 L CNN
+F 2 "Capacitor_SMD:C_0805_2012Metric_Pad1.15x1.40mm_HandSolder" H 6438 1550 50  0001 C CNN
+F 3 "~" H 6400 1700 50  0001 C CNN
+	1    6400 1700
 	1    0    0    -1
 $EndComp
@@
 L power:GND #PWR0128
 U 1 1 5EFA5875
-P 8350 1950
-F 0 "#PWR0128" H 8350 1700 50  0001 C CNN
-F 1 "GND" H 8355 1777 50  0000 C CNN
-F 2 "" H 8350 1950 50  0001 C CNN
-F 3 "" H 8350 1950 50  0001 C CNN
-	1    8350 1950
-	1    0    0    -1
-$EndComp
-Connection ~ 8350 1650
+P 6400 1850
+F 0 "#PWR0128" H 6400 1600 50  0001 C CNN
+F 1 "GND" H 6405 1677 50  0000 C CNN
+F 2 "" H 6400 1850 50  0001 C CNN
+F 3 "" H 6400 1850 50  0001 C CNN
+	1    6400 1850
+	1    0    0    -1
+$EndComp
 $Comp
 L Device:C C2
@@
 L Amplifier_Operational:TL072 U1
 U 1 1 5EE9233E
-P 6850 1650
-F 0 "U1" H 6850 2017 50  0000 C CNN
-F 1 "TL072" H 6850 1926 50  0000 C CNN
-F 2 "Package_SO:SOIC-8_3.9x4.9mm_P1.27mm" H 6850 1650 50  0001 C CNN
-F 3 "http://www.ti.com/lit/ds/symlink/tl071.pdf" H 6850 1650 50  0001 C CNN
-	1    6850 1650
-	1    0    0    -1
-$EndComp
-Wire Wire Line
-	6550 1550 6250 1550
-Wire Wire Line
-	6550 1750 6450 1750
-Wire Wire Line
-	6450 1750 6450 1950
-Wire Wire Line
-	6450 1950 7250 1950
-Wire Wire Line
-	7250 1950 7250 1650
-Wire Wire Line
-	7250 1650 7150 1650
-Connection ~ 7250 1650
+P 7750 1650
+F 0 "U1" H 7750 2017 50  0000 C CNN
+F 1 "TL072" H 7750 1926 50  0000 C CNN
+F 2 "Package_SO:SOIC-8_3.9x4.9mm_P1.27mm" H 7750 1650 50  0001 C CNN
+F 3 "http://www.ti.com/lit/ds/symlink/tl071.pdf" H 7750 1650 50  0001 C CNN
+	1    7750 1650
+	1    0    0    -1
+$EndComp
+Wire Wire Line
+	7450 1550 6400 1550
+Wire Wire Line
+	7450 1750 7350 1750
+Wire Wire Line
+	8150 1650 8050 1650
 $Comp
 L Amplifier_Operational:TL072 U1
@@
 L power:+12V #PWR0126
 U 1 1 5EE80416
-P 8500 2850
-F 0 "#PWR0126" H 8500 2700 50  0001 C CNN
-F 1 "+12V" V 8515 2978 50  0000 L CNN
-F 2 "" H 8500 2850 50  0001 C CNN
-F 3 "" H 8500 2850 50  0001 C CNN
-	1    8500 2850
+P 10150 4100
+F 0 "#PWR0126" H 10150 3950 50  0001 C CNN
+F 1 "+12V" V 10165 4228 50  0000 L CNN
+F 2 "" H 10150 4100 50  0001 C CNN
+F 3 "" H 10150 4100 50  0001 C CNN
+	1    10150 4100
 	0    -1   -1   0
 $EndComp
-Connection ~ 8500 2850
+Connection ~ 10150 4100
 $Comp
 L power:-12V #PWR0127
 U 1 1 5EE80C0B
-P 8500 3250
-F 0 "#PWR0127" H 8500 3350 50  0001 C CNN
-F 1 "-12V" V 8515 3378 50  0000 L CNN
-F 2 "" H 8500 3250 50  0001 C CNN
-F 3 "" H 8500 3250 50  0001 C CNN
-	1    8500 3250
+P 10150 4500
+F 0 "#PWR0127" H 10150 4600 50  0001 C CNN
+F 1 "-12V" V 10165 4628 50  0000 L CNN
+F 2 "" H 10150 4500 50  0001 C CNN
+F 3 "" H 10150 4500 50  0001 C CNN
+	1    10150 4500
 	0    -1   -1   0
 $EndComp
-Connection ~ 8500 3250
+Connection ~ 10150 4500
 $Comp
 L power:-12V #PWR0131
@@
 	1    0    0    -1
 $EndComp
+Connection ~ 8150 1650
+Connection ~ 6400 1550
+Wire Wire Line
+	6400 1550 6250 1550
+$Comp
+L power:GND #PWR0139
+U 1 1 5EF10DFE
+P 7350 2400
+F 0 "#PWR0139" H 7350 2150 50  0001 C CNN
+F 1 "GND" H 7355 2227 50  0000 C CNN
+F 2 "" H 7350 2400 50  0001 C CNN
+F 3 "" H 7350 2400 50  0001 C CNN
+	1    7350 2400
+	1    0    0    -1
+$EndComp
+Wire Wire Line
+	7350 1750 7350 2000
+Wire Wire Line
+	7350 2000 7600 2000
+Connection ~ 7350 2000
+Wire Wire Line
+	7350 2000 7350 2100
+Wire Wire Line
+	7900 2000 8150 2000
+Wire Wire Line
+	8150 1650 8150 2000
+Wire Wire Line
+	7750 2150 7750 2250
+Wire Wire Line
+	7750 2250 8150 2250
+Wire Wire Line
+	8150 2250 8150 2000
+Connection ~ 8150 2000
+Text Notes 7500 2350 0    50   ~ 0
+octave switch trim
+$Comp
+L Connector:TestPoint TP2
+U 1 1 5EF4A910
+P 8350 1150
+F 0 "TP2" H 8408 1268 50  0000 L CNN
+F 1 "TestPoint" H 8408 1177 50  0000 L CNN
+F 2 "TestPoint:TestPoint_Keystone_5000-5004_Miniature" H 8550 1150 50  0001 C CNN
+F 3 "~" H 8550 1150 50  0001 C CNN
+	1    8350 1150
+	1    0    0    -1
+$EndComp
+Connection ~ 8350 1150
+$Comp
+L Connector:TestPoint TP1
+U 1 1 5EF4CA65
+P 8350 750
+F 0 "TP1" H 8408 868 50  0000 L CNN
+F 1 "TestPoint" H 8408 777 50  0000 L CNN
+F 2 "TestPoint:TestPoint_Keystone_5000-5004_Miniature" H 8550 750 50  0001 C CNN
+F 3 "~" H 8550 750 50  0001 C CNN
+	1    8350 750
+	1    0    0    -1
+$EndComp
+$Comp
+L power:GND #PWR05
+U 1 1 5EF4D264
+P 8350 750
+F 0 "#PWR05" H 8350 500 50  0001 C CNN
+F 1 "GND" H 8355 577 50  0000 C CNN
+F 2 "" H 8350 750 50  0001 C CNN
+F 3 "" H 8350 750 50  0001 C CNN
+	1    8350 750
+	1    0    0    -1
+$EndComp
