File: new_stuff_june_2020/oscillator_carrier_board/kicad_docs/aux_waveshaper_components.sch (KiCad schematic (older format))
At the start: 5 parts, among them J11 Conn_01x05, J12 Conn_01x03, J13 power_header

Commit message: make gerbers of most boards, add unfinished modulation source
Other:
- moved on the sheet: J11, J12, J13
Changed lines of the file:
@@
 L Connector_Generic:Conn_02x05_Odd_Even J?
 U 1 1 5EFB3359
-P 5300 4200
+P 5600 4600
 AR Path="/5EFB3359" Ref="J?"  Part="1"
 AR Path="/5EF50E5A/5EFB3359" Ref="J?"  Part="1"
 AR Path="/5EFAF067/5EFB3359" Ref="J13"  Part="1"
-F 0 "J13" H 5250 3750 50  0000 C CNN
-F 1 "power_header" H 5200 3850 50  0000 C CNN
-F 2 "Connector_PinSocket_2.54mm:PinSocket_2x05_P2.54mm_Vertical" H 5300 4200 50  0001 C CNN
-F 3 "~" H 5300 4200 50  0001 C CNN
-	1    5300 4200
+F 0 "J13" H 5550 4150 50  0000 C CNN
+F 1 "power_header" H 5500 4250 50  0000 C CNN
+F 2 "Connector_PinSocket_2.54mm:PinSocket_2x05_P2.54mm_Vertical" H 5600 4600 50  0001 C CNN
+F 3 "~" H 5600 4600 50  0001 C CNN
+	1    5600 4600
 	-1   0    0    1
 $EndComp
 Wire Wire Line
-	5000 4000 5500 4000
+	5300 4400 5800 4400
 Wire Wire Line
-	5500 4100 5500 4200
+	5800 4500 5800 4600
 Wire Wire Line
-	5500 4200 5500 4300
-Connection ~ 5500 4200
+	5800 4600 5800 4700
+Connection ~ 5800 4600
 Wire Wire Line
-	5500 4300 5000 4300
-Connection ~ 5500 4300
+	5800 4700 5300 4700
+Connection ~ 5800 4700
 Wire Wire Line
-	5000 4300 5000 4200
-Connection ~ 5000 4300
+	5300 4700 5300 4600
+Connection ~ 5300 4700
 Wire Wire Line
-	5000 4200 5000 4100
-Connection ~ 5000 4200
+	5300 4600 5300 4500
+Connection ~ 5300 4600
 Wire Wire Line
-	5000 4100 5500 4100
-Connection ~ 5000 4100
-Connection ~ 5500 4100
+	5300 4500 5800 4500
+Connection ~ 5300 4500
+Connection ~ 5800 4500
 Wire Wire Line
-	5500 4200 5000 4200
+	5800 4600 5300 4600
 Wire Wire Line
-	5000 4400 5500 4400
+	5300 4800 5800 4800
 $Comp
 L power:GND #PWR?
 U 1 1 5EFB336E
-P 5000 4200
+P 5300 4600
 AR Path="/5EF50E5A/5EFB336E" Ref="#PWR?"  Part="1"
 AR Path="/5EFAF067/5EFB336E" Ref="#PWR0130"  Part="1"
-F 0 "#PWR0130" H 5000 3950 50  0001 C CNN
-F 1 "GND" V 5005 4072 50  0000 R CNN
-F 2 "" H 5000 4200 50  0001 C CNN
-F 3 "" H 5000 4200 50  0001 C CNN
-	1    5000 4200
+F 0 "#PWR0130" H 5300 4350 50  0001 C CNN
+F 1 "GND" V 5305 4472 50  0000 R CNN
+F 2 "" H 5300 4600 50  0001 C CNN
+F 3 "" H 5300 4600 50  0001 C CNN
+	1    5300 4600
 	0    1    1    0
 $EndComp
 Wire Wire Line
-	2750 2300 2850 2300
+	5200 2200 5300 2200
 Wire Wire Line
-	2750 2400 2750 2300
+	5200 2300 5200 2200
 $Comp
 L power:GND #PWR?
 U 1 1 5EFB48BF
-P 2750 2400
+P 5200 2300
 AR Path="/5EFB48BF" Ref="#PWR?"  Part="1"
 AR Path="/5EFAF067/5EFB48BF" Ref="#PWR0133"  Part="1"
-F 0 "#PWR0133" H 2750 2150 50  0001 C CNN
-F 1 "GND" H 2755 2227 50  0000 C CNN
-F 2 "" H 2750 2400 50  0001 C CNN
-F 3 "" H 2750 2400 50  0001 C CNN
-	1    2750 2400
+F 0 "#PWR0133" H 5200 2050 50  0001 C CNN
+F 1 "GND" H 5205 2127 50  0000 C CNN
+F 2 "" H 5200 2300 50  0001 C CNN
+F 3 "" H 5200 2300 50  0001 C CNN
+	1    5200 2300
 	1    0    0    -1
 $EndComp
@@
 L Connector_Generic:Conn_01x05 J?
 U 1 1 5EFB48B5
-P 3050 2100
+P 5500 2000
 AR Path="/5EFB48B5" Ref="J?"  Part="1"
 AR Path="/5EFAF067/5EFB48B5" Ref="J11"  Part="1"
-F 0 "J11" H 3130 2142 50  0000 L CNN
-F 1 "Conn_01x05" H 3130 2051 50  0000 L CNN
-F 2 "Connector_PinSocket_2.54mm:PinSocket_1x05_P2.54mm_Vertical" H 3050 2100 50  0001 C CNN
-F 3 "~" H 3050 2100 50  0001 C CNN
-	1    3050 2100
+F 0 "J11" H 5580 2042 50  0000 L CNN
+F 1 "Conn_01x05" H 5580 1951 50  0000 L CNN
+F 2 "Connector_PinSocket_2.54mm:PinSocket_1x05_P2.54mm_Vertical" H 5500 2000 50  0001 C CNN
+F 3 "~" H 5500 2000 50  0001 C CNN
+	1    5500 2000
 	1    0    0    -1
 $EndComp
-Text HLabel 2850 1900 0    50   Input ~ 0
+Text HLabel 5300 1800 0    50   Input ~ 0
 sine_in
-Text HLabel 2850 2000 0    50   Input ~ 0
+Text HLabel 5300 1900 0    50   Input ~ 0
 tri_in
-Text HLabel 2850 2100 0    50   Input ~ 0
+Text HLabel 5300 2000 0    50   Input ~ 0
 saw_in
-Text HLabel 2850 2200 0    50   Input ~ 0
+Text HLabel 5300 2100 0    50   Input ~ 0
 pulse_in
 $Comp
 L Connector_Generic:Conn_01x03 J12
 U 1 1 5EFBC485
-P 3100 3250
-F 0 "J12" H 3180 3292 50  0000 L CNN
-F 1 "Conn_01x03" H 3180 3201 50  0000 L CNN
-F 2 "Connector_PinSocket_2.54mm:PinSocket_1x03_P2.54mm_Vertical" H 3100 3250 50  0001 C CNN
-F 3 "~" H 3100 3250 50  0001 C CNN
-	1    3100 3250
+P 5550 3150
+F 0 "J12" H 5630 3192 50  0000 L CNN
+F 1 "Conn_01x03" H 5630 3101 50  0000 L CNN
+F 2 "Connector_PinSocket_2.54mm:PinSocket_1x03_P2.54mm_Vertical" H 5550 3150 50  0001 C CNN
+F 3 "~" H 5550 3150 50  0001 C CNN
+	1    5550 3150
 	1    0    0    -1
 $EndComp
-Text HLabel 2900 3150 0    50   Input ~ 0
+Text HLabel 5350 3050 0    50   Input ~ 0
 man_pulse_in
-Text HLabel 2900 3250 0    50   Input ~ 0
+Text HLabel 5350 3150 0    50   Input ~ 0
 PWM_in
 Wire Wire Line
-	2800 3350 2900 3350
+	5250 3250 5350 3250
 Wire Wire Line
-	2800 3450 2800 3350
+	5250 3350 5250 3250
 $Comp
 L power:GND #PWR?
 U 1 1 5EFBD5ED
-P 2800 3450
+P 5250 3350
 AR Path="/5EFBD5ED" Ref="#PWR?"  Part="1"
 AR Path="/5EFAF067/5EFBD5ED" Ref="#PWR0134"  Part="1"
-F 0 "#PWR0134" H 2800 3200 50  0001 C CNN
-F 1 "GND" H 2805 3277 50  0000 C CNN
-F 2 "" H 2800 3450 50  0001 C CNN
-F 3 "" H 2800 3450 50  0001 C CNN
-	1    2800 3450
+F 0 "#PWR0134" H 5250 3100 50  0001 C CNN
+F 1 "GND" H 5255 3177 50  0000 C CNN
+F 2 "" H 5250 3350 50  0001 C CNN
+F 3 "" H 5250 3350 50  0001 C CNN
+	1    5250 3350
 	1    0    0    -1
 $EndComp
@@
 L power:+12V #PWR0137
 U 1 1 5EE889ED
-P 5000 4000
-F 0 "#PWR0137" H 5000 3850 50  0001 C CNN
-F 1 "+12V" V 5015 4128 50  0000 L CNN
-F 2 "" H 5000 4000 50  0001 C CNN
-F 3 "" H 5000 4000 50  0001 C CNN
-	1    5000 4000
+P 5300 4400
+F 0 "#PWR0137" H 5300 4250 50  0001 C CNN
+F 1 "+12V" V 5315 4528 50  0000 L CNN
+F 2 "" H 5300 4400 50  0001 C CNN
+F 3 "" H 5300 4400 50  0001 C CNN
+	1    5300 4400
 	0    -1   -1   0
 $EndComp
-Connection ~ 5000 4000
+Connection ~ 5300 4400
 $Comp
 L power:-12V #PWR0138
 U 1 1 5EE8902A
-P 5000 4400
-F 0 "#PWR0138" H 5000 4500 50  0001 C CNN
-F 1 "-12V" V 5015 4528 50  0000 L CNN
-F 2 "" H 5000 4400 50  0001 C CNN
-F 3 "" H 5000 4400 50  0001 C CNN
-	1    5000 4400
+P 5300 4800
+F 0 "#PWR0138" H 5300 4900 50  0001 C CNN
+F 1 "-12V" V 5315 4928 50  0000 L CNN
+F 2 "" H 5300 4800 50  0001 C CNN
+F 3 "" H 5300 4800 50  0001 C CNN
+	1    5300 4800
 	0    -1   -1   0
 $EndComp
-Connection ~ 5000 4400
+Connection ~ 5300 4800
 $EndSCHEMATC
