File: new_stuff_june_2020/oscillator_carrier_board/kicad_docs/oscillator_carrier_board.kicad_pcb (KiCad board)
At the start: 2 copper layers, 99.1 x 99.1 mm, 36 parts, among them J1 Conn_01x06, J10 Conn_01x05, J11 Conn_01x05, J12 Conn_01x03, J13 power_header, J2 Conn_01x05, J3 power_header, J4 Conn_01x04, J5 Conn_01x02, J6 Conn_01x02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

Commit message: make gerbers of most boards, add unfinished modulation source
Parts:
- added TP1: TestPoint, TestPoint:TestPoint_Keystone_5000-5004_Miniature, F.Cu at (124.5, 144.8)
- added TP2: TestPoint, TestPoint:TestPoint_Keystone_5000-5004_Miniature, F.Cu at (124.5, 134.6)
- SW1: value SW_Rotary12 -> octave_switch
- moved R7 21.8 mm to (114.5, 86.1), turned to 180 degrees
- moved C1 20.3 mm to (130.6, 59.7)
Connections:
- J10 pad 1: Net-(C1-Pad1) -> Net-(J10-Pad1)
- R7 pad 1: Net-(C1-Pad1) -> Net-(R7-Pad1)
- R7 pad 2: Net-(R7-Pad2) -> GND
- RV6 pad 1: Net-(R7-Pad2) -> Net-(R7-Pad1)
- RV6 pad 2: Net-(R7-Pad2) -> Net-(J10-Pad1)
- RV6 pad 3: Net-(RV6-Pad3) -> Net-(J10-Pad1)
- SW1 pad 13: Net-(SW1-Pad13) -> Net-(C1-Pad1)
- U1 pad 1: Net-(RV6-Pad3) -> Net-(J10-Pad1)
- U1 pad 2: Net-(RV6-Pad3) -> Net-(R7-Pad1)
- U1 pad 3: Net-(SW1-Pad13) -> Net-(C1-Pad1)
Routing:
- net Net-(J10-Pad1): track 0.00 -> 103.4 mm, vias 0 -> 2
- net Net-(R7-Pad2): track 86.5 -> 0.00 mm
- net Net-(R7-Pad1): track 0.00 -> 67.0 mm
- net Net-(RV6-Pad3): track 57.8 -> 0.00 mm
- net Net-(SW1-Pad13): track 29.5 -> 0.00 mm
- net Net-(C1-Pad1): track 8.89 -> 32.7 mm
- net /VCO_core_components/sync_in: track 131.4 -> 138.3 mm
- net GND: vias 28 -> 27
Other:
- board text added: "octave switch test point"
