File: new_stuff_june_2020/dual_ADSR/dual_ADSR_carrier_board/kicad_docs/opamp_LPFs.sch (KiCad schematic (older format))
At the start: 26 parts, among them U1 TL072, U2 TL072

Commit message: add component values to ADSR LPFs
Parts:
- C15, C16, C17, C18: value C -> 2n2
- R10, R9: value R -> 50k
- R11, R12: value R -> 200k
- R13, R14: value R -> 33k
- R15, R16: value R -> 68k
Changed lines of the file:
@@
 P 5450 2200
 F 0 "R15" V 5550 2200 50  0000 C CNN
-F 1 "R" V 5450 2200 50  0000 C CNN
+F 1 "68k" V 5450 2200 50  0000 C CNN
 F 2 "Resistor_SMD:R_0805_2012Metric_Pad1.15x1.40mm_HandSolder" V 5380 2200 50  0001 C CNN
 F 3 "~" H 5450 2200 50  0001 C CNN
@@
 P 5050 2450
 F 0 "R13" H 5200 2450 50  0000 C CNN
-F 1 "R" V 5050 2450 50  0000 C CNN
+F 1 "33k" V 5050 2450 50  0000 C CNN
 F 2 "Resistor_SMD:R_0805_2012Metric_Pad1.15x1.40mm_HandSolder" V 4980 2450 50  0001 C CNN
 F 3 "~" H 5050 2450 50  0001 C CNN
@@
 P 4450 1750
 F 0 "R11" V 4550 1750 50  0000 C CNN
-F 1 "R" V 4450 1750 50  0000 C CNN
+F 1 "200k" V 4450 1750 50  0000 C CNN
 F 2 "Resistor_SMD:R_0805_2012Metric_Pad1.15x1.40mm_HandSolder" V 4380 1750 50  0001 C CNN
 F 3 "~" H 4450 1750 50  0001 C CNN
@@
 P 4700 2000
 F 0 "C17" H 4815 2046 50  0000 L CNN
-F 1 "C" H 4815 1955 50  0000 L CNN
+F 1 "2n2" H 4815 1955 50  0000 L CNN
 F 2 "Capacitor_SMD:C_0805_2012Metric_Pad1.15x1.40mm_HandSolder" H 4738 1850 50  0001 C CNN
 F 3 "~" H 4700 2000 50  0001 C CNN
@@
 P 4450 1350
 F 0 "C15" V 4198 1350 50  0000 C CNN
-F 1 "C" V 4289 1350 50  0000 C CNN
+F 1 "2n2" V 4289 1350 50  0000 C CNN
 F 2 "Capacitor_SMD:C_0805_2012Metric_Pad1.15x1.40mm_HandSolder" H 4488 1200 50  0001 C CNN
 F 3 "~" H 4450 1350 50  0001 C CNN
@@
 P 3950 1750
 F 0 "R9" V 4050 1750 50  0000 C CNN
-F 1 "R" V 3950 1750 50  0000 C CNN
+F 1 "50k" V 3950 1750 50  0000 C CNN
 F 2 "Resistor_SMD:R_0805_2012Metric_Pad1.15x1.40mm_HandSolder" V 3880 1750 50  0001 C CNN
 F 3 "~" H 3950 1750 50  0001 C CNN
@@
 P 5450 4650
 F 0 "R16" V 5550 4650 50  0000 C CNN
-F 1 "R" V 5450 4650 50  0000 C CNN
+F 1 "68k" V 5450 4650 50  0000 C CNN
 F 2 "Resistor_SMD:R_0805_2012Metric_Pad1.15x1.40mm_HandSolder" V 5380 4650 50  0001 C CNN
 F 3 "~" H 5450 4650 50  0001 C CNN
@@
 P 5050 4900
 F 0 "R14" H 5200 4900 50  0000 C CNN
-F 1 "R" V 5050 4900 50  0000 C CNN
+F 1 "33k" V 5050 4900 50  0000 C CNN
 F 2 "Resistor_SMD:R_0805_2012Metric_Pad1.15x1.40mm_HandSolder" V 4980 4900 50  0001 C CNN
 F 3 "~" H 5050 4900 50  0001 C CNN
@@
 P 4450 4200
 F 0 "R12" V 4550 4200 50  0000 C CNN
-F 1 "R" V 4450 4200 50  0000 C CNN
+F 1 "200k" V 4450 4200 50  0000 C CNN
 F 2 "Resistor_SMD:R_0805_2012Metric_Pad1.15x1.40mm_HandSolder" V 4380 4200 50  0001 C CNN
 F 3 "~" H 4450 4200 50  0001 C CNN
@@
 P 4700 4450
 F 0 "C18" H 4815 4496 50  0000 L CNN
-F 1 "C" H 4815 4405 50  0000 L CNN
+F 1 "2n2" H 4815 4405 50  0000 L CNN
 F 2 "Capacitor_SMD:C_0805_2012Metric_Pad1.15x1.40mm_HandSolder" H 4738 4300 50  0001 C CNN
 F 3 "~" H 4700 4450 50  0001 C CNN
@@
 P 4450 3800
 F 0 "C16" V 4198 3800 50  0000 C CNN
-F 1 "C" V 4289 3800 50  0000 C CNN
+F 1 "2n2" V 4289 3800 50  0000 C CNN
 F 2 "Capacitor_SMD:C_0805_2012Metric_Pad1.15x1.40mm_HandSolder" H 4488 3650 50  0001 C CNN
 F 3 "~" H 4450 3800 50  0001 C CNN
@@
 P 3950 4200
 F 0 "R10" V 4050 4200 50  0000 C CNN
-F 1 "R" V 3950 4200 50  0000 C CNN
+F 1 "50k" V 3950 4200 50  0000 C CNN
 F 2 "Resistor_SMD:R_0805_2012Metric_Pad1.15x1.40mm_HandSolder" V 3880 4200 50  0001 C CNN
 F 3 "~" H 3950 4200 50  0001 C CNN
