File: new_stuff_june_2020/dual_ADSR/dual_ADSR_carrier_board/kicad_docs/dual_ADSR.kicad_pcb (KiCad board)
At the start: 2 copper layers, 99.1 x 133.3 mm, 71 parts, among them J1 inputs, J2 power_in, J3 outputs, J4 stm32_DC_in, J5 3.3v, J6 gnd, J7 port_A, J8 port_B, J9 port_C, Q1 MMBT3904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

Commit message: add values to pcb, regenerate BOM
Parts:
- C15, C16, C17, C18: value C -> 2n2
- R10, R9: value R -> 50k
- R11, R12: value R -> 200k
- R13, R14: value R -> 33k
- R15, R16: value R -> 68k
