File: new_stuff_june_2020/dual_VCA/kicad_docs/dual_VCA.kicad_pcb (KiCad board)
At the start: 2 copper layers, 99.1 x 99.1 mm, 70 parts, among them J1 VCA_1_port, J2 VCA_2_port, J7 power_input, U1 SSM2164, U2 TL072, U3 TL072, U4 TL072, U5 TL072, U6 MAX6035xxUR50

Commit message: generate BOMs for most boards
Parts:
- R23: value R -> opt
- RV5, RV6: value 100k -> 10k
