File: new_stuff_june_2020/CEM3340_VCO/kicad_docs/CEM3340_VCO.kicad_pcb (KiCad board)
At the start: 2 copper layers, 55.9 x 78.7 mm, 96 parts, among them J1 tuning controls, J2 1 v/oct inputs, J3 linear FM input, J4 sync input, J5 PWM inputs, J6 power input, Q1 MMDT3904, U1 L78L10_SOT89, U2 MC7905, U3 REF02AU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

Commit message: fill in VCO r values, generate BOM
Parts:
- removed hole 1: MountingHole_3.2mm_M3, MountingHole:MountingHole_3.2mm_M3
- removed hole 2: MountingHole_3.2mm_M3, MountingHole:MountingHole_3.2mm_M3
- added H1: MountingHole, MountingHole:MountingHole_3.2mm_M3, F.Cu at (81.3, 55.9)
- added H2: MountingHole, MountingHole:MountingHole_3.2mm_M3, F.Cu at (81.3, 124.5)
- C12: value C -> 100nF
- R30: value ??? -> 34k
- R32: value ??? -> 68k
- R35, R36: value 11k -> 15k
- R4: value ??? -> 1M
- R40, R44: value R -> 2k
- R5: value ??? -> 100k
- R6: value 270k -> 110k
