File: new_stuff_june_2020/four_pole_lpf/four_pole_lpf.sch (KiCad schematic (older format))
At the start: 35 parts, among them Q1 BC850, Q2 BC860, U1 SSM2164, U2 TL072, U3 TL072, U4 TL072

Commit message: mess around with 2164 lpf
Parts:
- removed C1: 3n3, symbol Device:C
- removed C2, C4, C6, C8: 220pF, symbol Device:C
- removed C3, C5, C7: 5n6, symbol Device:C
- removed D1, D2: 1N914WT, Diode_SMD:D_SOD-523, symbol Diode:1N914WT
- removed Q1: BC850, Package_TO_SOT_SMD:SOT-23, symbol Transistor_BJT:BC850
- removed Q2: BC860, Package_TO_SOT_SMD:SOT-23, symbol Transistor_BJT:BC860
- removed R1, R10, R13, R15, R16, R18, R3, R7: 15k, symbol Device:R
- removed R11, R12: 10k, symbol Device:R
- removed R14, R17, R9: 180, symbol Device:R
- removed R2: 75, symbol Device:R
- removed R4: 5k49, symbol Device:R
- removed R5: ???, symbol Device:R
- removed R6, R8: 510, symbol Device:R
- removed RV1: 10k, symbol Device:R_POT
- removed U1: SSM2164, symbol lpf_parts:SSM2164
- removed U2, U3, U4: TL072, symbol Amplifier_Operational:TL072
Other:
- note removed: "resonance"
