File: new_stuff_june_2020/five_pulser_board/kicad_docs/five_pulser_board.sch (KiCad schematic (older format))
At the start: 49 parts, among them J1 signal_in, J2 CV_in, J3 Conn_02x05_Odd_Even, J4 signal_out, J5 pulses, U1 TL072, U2 LM3914, U3 TL072

Commit message: fix pcb error, change some values
Parts:
- C7: value 56pF -> 100nF
- R2, R7: value 220k -> 100k
- R3, R9: value 22k -> 10k
- R4: value 200k -> 100k
- R5, R6, R8: value 82k -> 100k

Commit message: scale pwm circuit and add power flags
Parts:
- R8: value 100k -> 39k
Connections:
- no-connect marks 8 -> 9
Changed lines of the file:
@@
 P 2900 3000
 F 0 "R8" V 2800 3000 50  0000 C CNN
-F 1 "100k" V 2900 3000 50  0000 C CNN
+F 1 "39k" V 2900 3000 50  0000 C CNN
 F 2 "Resistor_SMD:R_0805_2012Metric_Pad1.15x1.40mm_HandSolder" V 2830 3000 50  0001 C CNN
 F 3 "~" H 2900 3000 50  0001 C CNN
@@
 	0    1    1    0
 $EndComp
+NoConn ~ 4750 1550
+$Comp
+L power:PWR_FLAG #FLG0101
+U 1 1 5F03A7F6
+P 1650 5150
+F 0 "#FLG0101" H 1650 5225 50  0001 C CNN
+F 1 "PWR_FLAG" V 1650 5278 50  0000 L CNN
+F 2 "" H 1650 5150 50  0001 C CNN
+F 3 "~" H 1650 5150 50  0001 C CNN
+	1    1650 5150
+	0    1    1    0
+$EndComp
+Connection ~ 1650 5150
+$Comp
+L power:PWR_FLAG #FLG0102
+U 1 1 5F03BA1F
+P 1650 5350
+F 0 "#FLG0102" H 1650 5425 50  0001 C CNN
+F 1 "PWR_FLAG" V 1650 5478 50  0000 L CNN
+F 2 "" H 1650 5350 50  0001 C CNN
+F 3 "~" H 1650 5350 50  0001 C CNN
+	1    1650 5350
+	0    1    1    0
+$EndComp
+$Comp
+L power:PWR_FLAG #FLG0103
+U 1 1 5F03BBB2
+P 1650 5550
+F 0 "#FLG0103" H 1650 5625 50  0001 C CNN
+F 1 "PWR_FLAG" V 1650 5678 50  0000 L CNN
+F 2 "" H 1650 5550 50  0001 C CNN
+F 3 "~" H 1650 5550 50  0001 C CNN
+	1    1650 5550
+	0    1    1    0
+$EndComp
+Connection ~ 1650 5550
 $EndSCHEMATC
