File: new_stuff_june_2020/sub_osc_board/kicad_docs/sub_osc_board.sch (KiCad schematic (older format))
At the start: 25 parts, among them J1 signal_inputs, J2 pwm_inputs, J4 signal_outputs, J5 Conn_01x03, J6 Conn_01x03, J7 Conn_01x03, U10 TL072, U6 TL072, U9 TL072

Commit message: change value to do-not-fit
Parts:
- R42: value 100k -> dnf
Changed lines of the file:
@@
 P 2500 4850
 F 0 "R42" H 2350 4850 50  0000 C CNN
-F 1 "100k" V 2500 4850 50  0000 C CNN
+F 1 "dnf" V 2500 4850 50  0000 C CNN
 F 2 "Resistor_SMD:R_0805_2012Metric_Pad1.15x1.40mm_HandSolder" V 2430 4850 50  0001 C CNN
 F 3 "~" H 2500 4850 50  0001 C CNN
