File: new_stuff_june_2020/sub_osc_board/kicad_docs/sub_osc_board.kicad_pcb (KiCad board)
At the start: 2 copper layers, 39.4 x 78.7 mm, 86 parts, among them J1 Conn_01x05, J2 Conn_01x03, J3 Conn_02x05_Odd_Even, J4 Conn_01x05, J5 Conn_01x03, J6 Conn_01x03, J7 Conn_01x03, Q1 MMBF4391, Q2 MMBF4391, Q3 MMBF4391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

Commit message: update pcb and BOM with correct values
Parts:
- J1: value Conn_01x05 -> signal_inputs
- J2: value Conn_01x03 -> pwm_inputs
- J3: value Conn_02x05_Odd_Even -> power_input
- J4: value Conn_01x05 -> signal_outputs
- R34, R35, R36, R37: value ??? -> 100k

Commit message: change FETs and cap values
Parts:
- C1, C18: value 47pF -> 1nF
- Q1, Q2, Q3, Q4: value MMBF4391 -> MMBF5457

Commit message: apply componet change to pcb
Parts:
- R42: value 100k -> dnf
