File: wave_folder/kicad_docs/wave_folder.kicad_pcb (KiCad board)
At the start: 2 copper layers, 99.1 x 99.1 mm, 91 parts, among them J1 signal_port, J2 CV_port, J3 ring_mod_port, J4 power_in_connector, U1 SSM2164, U2 TL072, U3 TL072, U4 TL072, U5 AD534

Commit message: small changes to wave folder CV bias and output level
Parts:
- R12: value 10M -> dnf
- R21: value 56k -> 82k
