File: dual_MS20_VCF/kicad_docs/dual_MS20_VCF.kicad_pcb (KiCad board)
At the start: 2 copper layers, 99.1 x 99.1 mm, 91 parts, among them J1 Conn_01x05, J2 Conn_01x05, J3 power_in, J4 lpf_output_normal, Q1 BC558, Q2 BC558, Q3 BC558, Q4 BC558, U1 LM13700, U2 MC1458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

Commit message: change scaling resistors for manual cutoff controls
Parts:
- R24, R6: value 100k -> 240k
