File: oscillator_carrier_board/kicad_docs/VCO_core_components.sch (KiCad schematic (older format))
At the start: 30 parts, among them J10 Conn_01x05, J4 Conn_01x04, J5 Conn_01x02, J6 Conn_01x02, J7 Conn_01x05, J8 power_header, J9 to_VCO_board, SW1 octave_switch, U1 TL072

Commit message: fill in values for octave switch, add VCO carrier BOM
Parts:
- R1, R2, R3, R4, R5, R6: value 10k -> 1k
- R7: value ??? -> 68k
- RV6: value ??? -> 50k
Other:
- note added: "use 0.5% tolerance or\nbetter for R1 through R6"
Changed lines of the file:
@@
 AR Path="/5EF50E5A/5EF665A7" Ref="R6"  Part="1"
 F 0 "R6" V 4850 750 50  0000 C CNN
-F 1 "10k" V 4900 950 50  0000 C CNN
+F 1 "1k" V 4900 950 50  0000 C CNN
 F 2 "Resistor_SMD:R_0805_2012Metric_Pad1.15x1.40mm_HandSolder" V 4830 950 50  0001 C CNN
 F 3 "~" H 4900 950 50  0001 C CNN
@@
 AR Path="/5EF50E5A/5EF665B5" Ref="R5"  Part="1"
 F 0 "R5" V 4450 850 50  0000 C CNN
-F 1 "10k" V 4500 1050 50  0000 C CNN
+F 1 "1k" V 4500 1050 50  0000 C CNN
 F 2 "Resistor_SMD:R_0805_2012Metric_Pad1.15x1.40mm_HandSolder" V 4430 1050 50  0001 C CNN
 F 3 "~" H 4500 1050 50  0001 C CNN
@@
 AR Path="/5EF50E5A/5EF665BB" Ref="R4"  Part="1"
 F 0 "R4" V 4050 950 50  0000 C CNN
-F 1 "10k" V 4100 1150 50  0000 C CNN
+F 1 "1k" V 4100 1150 50  0000 C CNN
 F 2 "Resistor_SMD:R_0805_2012Metric_Pad1.15x1.40mm_HandSolder" V 4030 1150 50  0001 C CNN
 F 3 "~" H 4100 1150 50  0001 C CNN
@@
 AR Path="/5EF50E5A/5EF665C4" Ref="R3"  Part="1"
 F 0 "R3" V 3650 1050 50  0000 C CNN
-F 1 "10k" V 3700 1250 50  0000 C CNN
+F 1 "1k" V 3700 1250 50  0000 C CNN
 F 2 "Resistor_SMD:R_0805_2012Metric_Pad1.15x1.40mm_HandSolder" V 3630 1250 50  0001 C CNN
 F 3 "~" H 3700 1250 50  0001 C CNN
@@
 AR Path="/5EF50E5A/5EF665CF" Ref="R2"  Part="1"
 F 0 "R2" V 3250 1150 50  0000 C CNN
-F 1 "10k" V 3300 1350 50  0000 C CNN
+F 1 "1k" V 3300 1350 50  0000 C CNN
 F 2 "Resistor_SMD:R_0805_2012Metric_Pad1.15x1.40mm_HandSolder" V 3230 1350 50  0001 C CNN
 F 3 "~" H 3300 1350 50  0001 C CNN
@@
 AR Path="/5EF50E5A/5EF665DA" Ref="R1"  Part="1"
 F 0 "R1" V 2850 1250 50  0000 C CNN
-F 1 "10k" V 2900 1450 50  0000 C CNN
+F 1 "1k" V 2900 1450 50  0000 C CNN
 F 2 "Resistor_SMD:R_0805_2012Metric_Pad1.15x1.40mm_HandSolder" V 2830 1450 50  0001 C CNN
 F 3 "~" H 2900 1450 50  0001 C CNN
@@
 AR Path="/5EF50E5A/5EF66615" Ref="RV6"  Part="1"
 F 0 "RV6" V 7635 2000 50  0000 C CNN
-F 1 "???" V 7750 2000 50  0000 C CNN
+F 1 "50k" V 7750 2000 50  0000 C CNN
 F 2 "Potentiometer_THT:Potentiometer_Bourns_3296W_Vertical" H 7750 2000 50  0001 C CNN
 F 3 "~" H 7750 2000 50  0001 C CNN
@@
 AR Path="/5EF50E5A/5EF66620" Ref="R7"  Part="1"
 F 0 "R7" H 7250 2250 50  0000 C CNN
-F 1 "???" V 7350 2250 50  0000 C CNN
+F 1 "68k" V 7350 2250 50  0000 C CNN
 F 2 "Resistor_SMD:R_0805_2012Metric_Pad1.15x1.40mm_HandSolder" V 7280 2250 50  0001 C CNN
 F 3 "~" H 7350 2250 50  0001 C CNN
@@
 	1    0    0    -1
 $EndComp
+Text Notes 3050 900  0    50   ~ 0
+use 0.5% tolerance or\nbetter for R1 through R6
 $EndSCHEMATC
