File: oscillator_carrier_board/kicad_docs/oscillator_carrier_board.kicad_pcb (KiCad board)
At the start: 2 copper layers, 99.1 x 99.1 mm, 38 parts, among them J1 Conn_01x06, J10 Conn_01x05, J11 Conn_01x05, J12 Conn_01x03, J13 power_header, J2 Conn_01x05, J3 power_header, J4 Conn_01x04, J5 Conn_01x02, J6 Conn_01x02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

Commit message: fill in values for octave switch, add VCO carrier BOM
Parts:
- R1, R2, R3, R4, R5, R6: value 10k -> 1k
- R7: value ??? -> 68k
- RV6: value ??? -> 50k
