File: five_pulser_board/kicad_docs/five_pulser_board.kicad_pcb (KiCad board)
At the start: 2 copper layers, 39.4 x 78.7 mm, 49 parts, among them J1 signal_in, J2 CV_in, J3 Conn_02x05_Odd_Even, J4 signal_out, J5 pulses, U1 TL072, U2 LM3914, U3 TL072

Commit message: embiggen 5-pulser manual PW resistor
Parts:
- R4: value 100k -> 120k
