File: five_pulser_board/kicad_docs/five_pulser_board.sch (KiCad schematic (older format))
At the start: 49 parts, among them J1 signal_in, J2 CV_in, J3 Conn_02x05_Odd_Even, J4 signal_out, J5 pulses, U1 TL072, U2 LM3914, U3 TL072

Commit message: embiggen 5-pulser manual PW resistor
Parts:
- R4: value 100k -> 120k
Changed lines of the file:
@@
 P 2300 2750
 F 0 "R4" V 2200 2750 50  0000 C CNN
-F 1 "100k" V 2300 2750 50  0000 C CNN
+F 1 "120k" V 2300 2750 50  0000 C CNN
 F 2 "Resistor_SMD:R_0805_2012Metric_Pad1.15x1.40mm_HandSolder" V 2230 2750 50  0001 C CNN
 F 3 "~" H 2300 2750 50  0001 C CNN
