File: sub_osc_board/kicad_docs/sub_osc_board.kicad_pcb (KiCad board)
At the start: 2 copper layers, 39.4 x 78.7 mm, 86 parts, among them J1 signal_inputs, J2 pwm_inputs, J3 power_input, J4 signal_outputs, J5 Conn_01x03, J6 Conn_01x03, J7 Conn_01x03, Q1 MMBF5457, Q2 MMBF5457, Q3 MMBF5457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

Commit message: change sub-osc PWM range and mixer gain
Parts:
- R37: value 100k -> 33k
- R5: value 330k -> 110k
- R8: value 150k -> 100k
