File: circuit_boards/modulation_source/kicad_docs/modulation_source.kicad_pcb (KiCad board)
At the start: 2 copper layers, 99.1 x 68.6 mm, 73 parts, among them J1 power_in, Q1 BC560, Q2 BC560, Q3 BF245A, Q4 BC550, Q5 BC550, Q6 BC550, U1 LM13700, U2 TL072, U3 TL072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

Commit message: change cap so noise biases quicker
Parts:
- C5: value 47uF -> 1uF
