File: circuit_boards/modulation_source/kicad_docs/modulation_source.sch (KiCad schematic (older format))
At the start: 73 parts, among them J1 power_in, Q1 BC560, Q2 BC560, Q3 BF245A, Q4 BC550, Q5 BC550, Q6 BC550, U1 LM13700, U2 TL072, U3 TL072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

Commit message: change cap so noise biases quicker
Parts:
- C5: value 47uF -> 1uF
Changed lines of the file:
@@
 P 5750 2400
 F 0 "C5" H 5865 2446 50  0000 L CNN
-F 1 "47uF" H 5865 2355 50  0000 L CNN
+F 1 "1uF" H 5865 2355 50  0000 L CNN
 F 2 "Capacitor_THT:CP_Radial_D6.3mm_P2.50mm" H 5750 2400 50  0001 C CNN
 F 3 "~" H 5750 2400 50  0001 C CNN
